File: BRC_RaspberryPI_Hat.kicad_sch (KiCad schematic)
At the start: 23 parts, among them J1 GPIO, U1 CAT24C256, U2 SN754410NE, U3 ADS1115IDGS, U4 SN754410NE, U5 SN754410NE

Commit message: naming changes + erc errors fixed
Parts:
- added C2, C3, C4, C5: 1000uF/25V, Capacitor_THT:CP_Radial_D10.0mm_P5.00mm, symbol Device:C_Polarized
- added J2, J4, J6, J8: Servo, Connector_PinHeader_2.54mm:PinHeader_1x03_P2.54mm_Vertical, symbol Connector_Generic:Conn_01x03
- added J3: ServoPower, TerminalBlock_Phoenix:TerminalBlock_Phoenix_MKDS-1,5-2-5.08_1x02_P5.08mm_Horizontal, symbol Connector_Generic:Conn_01x02
- added R2, R3, R4, R5: 330, Resistor_SMD:R_0805_2012Metric, symbol Device:R
- C1: footprint (none) -> Capacitor_SMD:C_0805_2012Metric
- Ceramic_C1, Ceramic_C2, Ceramic_C3: footprint Capacitor_THT:CP_Radial_D4.0mm_P1.50mm -> Capacitor_THT:C_Disc_D5.0mm_W2.5mm_P5.00mm
- Electro_C1: value 220micro -> 220uF/25V; footprint Capacitor_THT:CP_Radial_D4.0mm_P1.50mm -> Capacitor_THT:CP_Radial_D8.0mm_P3.50mm; symbol Device:C -> Device:C_Polarized
- JP1: footprint (none) -> Jumper:SolderJumper-2_P1.3mm_Open_RoundedPad1.0x1.5mm
- R1: footprint (none) -> Resistor_SMD:R_0805_2012Metric
- U1: footprint (none) -> Package_SO:SOIC-8_3.9x4.9mm_P1.27mm
Connections:
- net +12V: now also Ceramic_C1.2, Ceramic_C2.2, Ceramic_C3.2, Electro_C1.1, PowerSupply1.2 (Pin_2), U2.8 (VCC2), U4.8 (VCC2), U5.8 (VCC2)
- net +3.3V: now also C1.1, JP1.2 (B), R1.1, U1.8 (VCC)
- net GND: now also U1.1 (A0), U1.2 (A1), U1.3 (A2), U5.15 (4A), U5.7 (2A), C2.2, C3.2, C4.2, C5.2, J2.3 (Pin_3), J3.2 (Pin_2), J4.3 (Pin_3), J6.3 (Pin_3), J8.3 (Pin_3)
- net GPIO11/SPI0.SCLK: now also R5.2
- net GPIO22: now also R3.2
- net GPIO26: now also J1.37 (Pin_37), R2.2
- net GPIO2/SDA1: now also U3.1 (ADDR)
- net GPIO3/SCL1: no longer U3.1 (ADDR)
- net GPIO4/GPCLK0: now also R4.2
- net ID_SCL: now also U1.6 (SCL)
- net ID_SDA: now also R1.2, U1.5 (SDA)
- new net: J6.1 (Pin_1), R4.1
- new net: J4.1 (Pin_1), R3.1
- new net: J2.1 (Pin_1), R2.1
- new net: J8.1 (Pin_1), R5.1
- new net VSERVO: C2.1, C3.1, C4.1, C5.1, J2.2 (Pin_2), J3.1 (Pin_1), J4.2 (Pin_2), J6.2 (Pin_2), J8.2 (Pin_2)
- no-connect marks 8 -> 9
Other:
- note removed: "5V"
- note removed: "DR3"
- note removed: "DR4"
- note removed: "DR5"
- note removed: "DR6"
- note removed: "DR7"
- note removed: "GND"
- title: (none) -> BRC Raspberry Pi HAT
